File: CHOP_battery_ board/chop_battery_board/chop_battery_board.kicad_pcb (KiCad board)
At the start: 4 copper layers, 70.9 x 36.3 mm, 14 parts, among them J1 Barrel_Jack, J13 Li18650, J14 BatteryToMainBoard, SW1 SW_Slide_DPDT, U1 UA741CP

Commit message: PCB Final 5/24
Parts:
- moved J14 22.6 mm to (203.5, 121.8), turned to 90 degrees
- moved J13 5.50 mm to (160.5, 110.5), turned to 0 degrees
Routing:
- net GND: track 24.4 -> 51.2 mm
- net Net-(D2-A): track 34.5 -> 50.7 mm

Commit message: Battery board edit
Connections:
- J14 pad 1: GND -> Net-(D2-A)
- J14 pad 2: Net-(D2-A) -> GND
Routing:
- net GND: track 51.2 -> 45.1 mm
Changed lines of the file:
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@@
 			)
 		)
-		(property "Description" ""
+		(property "Description" "Generic connector, single row, 01x02, script generated (kicad-library-utils/schlib/autogen/connector/)"
 			(at 0 0 90)
 			(layer "B.Fab")
@@
 			(remove_unused_layers no)
 			(roundrect_rratio 0.147059)
-			(net 1 "GND")
+			(net 4 "Net-(D2-A)")
 			(pinfunction "Pin_1")
 			(pintype "passive")
@@
 			(layers "*.Cu" "*.Mask")
 			(remove_unused_layers no)
-			(net 4 "Net-(D2-A)")
+			(net 1 "GND")
 			(pinfunction "Pin_2")
 			(pintype "passive")
@@
 	)
 	(segment
+		(start 203.4675 115.4675)
+		(end 203.4675 119.25)
+		(width 0.25)
+		(layer "F.Cu")
+		(net 1)
+	)
+	(segment
 		(start 181.5 112)
 		(end 183.826 109.674)
@@
 	)
 	(segment
+		(start 173.675 113)
+		(end 174.675 112)
+		(width 0.25)
+		(layer "F.Cu")
+		(net 1)
+	)
+	(segment
+		(start 174.675 112)
+		(end 181.5 112)
+		(width 0.25)
+		(layer "F.Cu")
+		(net 1)
+	)
+	(segment
+		(start 197.674 109.674)
+		(end 203.4675 115.4675)
+		(width 0.25)
+		(layer "F.Cu")
+		(net 1)
+	)
+	(segment
 		(start 169.675 125.175)
 		(end 169.675 123.5)
@@
 	)
 	(segment
-		(start 173.675 113)
-		(end 174.675 112)
-		(width 0.25)
-		(layer "F.Cu")
-		(net 1)
-	)
-	(segment
 		(start 183.826 109.674)
 		(end 197.674 109.674)
@@
 	)
 	(segment
-		(start 205.25 121.75)
-		(end 203.4675 121.75)
-		(width 0.25)
-		(layer "F.Cu")
-		(net 1)
-	)
-	(segment
-		(start 174.675 112)
-		(end 181.5 112)
-		(width 0.25)
-		(layer "F.Cu")
-		(net 1)
-	)
-	(segment
 		(start 182.69 119.31)
 		(end 185.875 119.31)
@@
 		(start 170 125.5)
 		(end 169.675 125.175)
-		(width 0.25)
-		(layer "F.Cu")
-		(net 1)
-	)
-	(segment
-		(start 206.5 120.5)
-		(end 205.25 121.75)
-		(width 0.25)
-		(layer "F.Cu")
-		(net 1)
-	)
-	(segment
-		(start 197.674 109.674)
-		(end 206.5 118.5)
-		(width 0.25)
-		(layer "F.Cu")
-		(net 1)
-	)
-	(segment
-		(start 206.5 118.5)
-		(end 206.5 120.5)
 		(width 0.25)
 		(layer "F.Cu")
@@
 	)
 	(segment
-		(start 203.4675 117.5325)
-		(end 203.4675 119.25)
+		(start 190.5 111)
+		(end 201.25 121.75)
 		(width 0.25)
 		(layer "F.Cu")
@@
 	)
 	(segment
-		(start 183.5 111)
-		(end 197 111)
+		(start 175 117)
+		(end 177.5 117)
 		(width 0.25)
 		(layer "F.Cu")
@@
 	)
 	(segment
-		(start 203.5 117.5)
-		(end 203.4675 117.5325)
+		(start 177.5 117)
+		(end 183.5 111)
+		(width 0.25)
+		(layer "F.Cu")
+		(net 4)
+	)
+	(segment
+		(start 201.25 121.75)
+		(end 203.0165 121.75)
 		(width 0.25)
 		(layer "F.Cu")
@@
 	)
 	(segment
-		(start 177.5 117)
-		(end 183.5 111)
-		(width 0.25)
-		(layer "F.Cu")
-		(net 4)
-	)
-	(segment
-		(start 197 111)
-		(end 203.5 117.5)
-		(width 0.25)
-		(layer "F.Cu")
-		(net 4)
-	)
-	(segment
 		(start 175 117)
 		(end 172 120)
@@
 	)
 	(segment
-		(start 175 117)
-		(end 177.5 117)
-		(width 0.25)
-		(layer "F.Cu")
+		(start 183.5 111)
+		(end 190.5 111)
+		(width 0.25)
+		(layer "F.Cu")
