File: CHOP_battery_ board/chop_battery_board/chop_battery_board.kicad_pcb (KiCad board)
At the start: 4 copper layers, 70.9 x 36.3 mm, 14 parts, among them J1 Barrel_Jack, J13 Li18650, J14 BatteryToMainBoard, SW1 SW_Slide_DPDT, U1 UA741CP

Commit message: Gerber files
Parts:
- added R5: 100 Ohm, Resistor_SMD:R_0603_1608Metric, F.Cu at (150.7, 116.5)
- added R6: 100 Ohm, Resistor_SMD:R_0603_1608Metric, F.Cu at (150.7, 121.5)
- added R7: 0.9 Ohm, Resistor_SMD:R_0603_1608Metric, F.Cu at (150.7, 119.0)
- added R8: 680 Ohm, Resistor_SMD:R_0603_1608Metric, F.Cu at (157.5, 130.5)
- added R9: 680 Ohm, Resistor_SMD:R_0603_1608Metric, F.Cu at (196.2, 127.5)
- R4: value 300-500 Ohm -> 150 Ohm
Connections:
- D1 pad 1: Net-(U1-IN+) -> Net-(D1-Pad1)
- SW1 pad 3: Net-(U1-IN+) -> Net-(R5-Pad2)
- U1 pad 2: Net-(J13-Pin_2) -> Net-(U1-IN-)
Routing:
- net Net-(U1-IN-): track 0.00 -> 93.2 mm
- net Net-(D1-Pad1): track 0.00 -> 37.8 mm
- net Net-(D3-A): track 22.3 -> 50.5 mm
- net Net-(R5-Pad2): track 0.00 -> 12.6 mm
- net GND: track 45.1 -> 51.9 mm
- net Net-(J13-Pin_2): track 2.49 -> 0.00 mm, vias 1 -> 0
- net Net-(U1-IN+): track 51.3 -> 50.2 mm
