File: CHOP_Microcontroller_Board/microcontroller_board/chop_microcontroller_board.kicad_pcb (KiCad board)
At the start: 4 copper layers, 126.4 x 69.8 mm, 33 parts, among them J11 HEATER_SIGNAL_1, J12 POWER_HEAT, J14 BatteryToMainBoard, J2 OLED, J3 Encoder, J6 PFLOW, J7 DISC PUMP, J8 RTC, U1 Teensy4.1_Mounted, U2 U3V50F24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

Commit message: Gerber files
Parts:
- added R8: 4.7k, NYSEARCH:R_0603_1608Metric, F.Cu at (103.7, 121.5)
Connections:
- net /HL4_CS renamed /uPC_RTD_CS
- net /HL4_PWM_IN renamed /uPC_PWM_IN
- J11 pad 9: unconnected-(J11-Pin_9-Pad9) -> /uPC_RTD_DRDY
- U1 pad 25: unconnected-(U1-33_MCLK2-Pad25) -> /uPC_RTD_DRDY
Routing:
- net /uPC_RTD_DRDY: track 0.00 -> 36.8 mm
- net +3.3V: track 35.7 -> 39.0 mm
- net /SAFETY_CS: track 30.8 -> 29.2 mm
