File: CHOP_Microcontroller_Board/microcontroller_board/chop_microcontroller_board.kicad_sch (KiCad schematic)
At the start: 31 parts, among them J11 HEATER_SIGNAL_1, J12 POWER_HEAT, J14 BatteryToMainBoard, J2 OLED, J3 Encoder, J6 PFLOW, J7 DISC PUMP, U1 Teensy4.1_Mounted, U2 U3V50F24, U3 U3V50F12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

Commit message: PCB Final 5/24
Parts:
- added J8: RTC, Connector_PinHeader_2.54mm:PinHeader_1x05_P2.54mm_Vertical, symbol Connector_Generic:Conn_01x05
- added MK5: Mounting_Hole, MountingHole:MountingHole_3.2mm_M3, symbol Mechanical:MountingHole
- J6: footprint Connector_PinHeader_2.54mm:PinHeader_1x05_P2.54mm_Vertical -> Connector_Molex:Molex_Micro-Fit_3.0_43650-0500_1x05_P3.00mm_Horizontal
- R6: value 470k -> 4.7k
- R7: value 220k -> 2.2k
Connections:
- net +5V: now also J8.1 (Pin_1)
- net GNDREF: now also J8.2 (Pin_2)
- net SCL: now also J8.3 (Pin_3)
- net SDA: now also J8.4 (Pin_4)

Commit message: CHOP 3d models 5/30
Parts:
- J14: footprint Connector_JST:JST_PH_S3B-PH-K_1x03_P2.00mm_Horizontal -> Connector_JST:JST_PH_S2B-PH-K_1x02_P2.00mm_Horizontal; symbol Connector_Generic:Conn_01x03 -> Connector_Generic:Conn_01x02
- J2: footprint Connector_PinHeader_2.54mm:PinHeader_1x04_P2.54mm_Vertical -> chop_footprint_library:128x64OLED
Connections:
- net at U1.17 (25_A11_RX6_SDA2): no longer J14.3 (Pin_3)
Changed lines of the file:
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@@
 	(wire
 		(pts
-			(xy 43.18 77.47) (xy 48.26 77.47)
-		)
-		(stroke
-			(width 0)
-			(type default)
-		)
-	)
-	(wire
-		(pts
 			(xy 40.005 103.505) (xy 40.005 147.955)
 		)
@@
 	(wire
 		(pts
-			(xy 114.3 72.39) (xy 114.3 92.71)
-		)
-		(stroke
-			(width 0)
-			(type default)
-		)
-	)
-	(wire
-		(pts
 			(xy 16.51 27.305) (xy 23.495 27.305)
 		)
@@
 	(wire
 		(pts
-			(xy 114.3 92.71) (xy 132.08 92.71)
-		)
-		(stroke
-			(width 0)
-			(type default)
-		)
-	)
-	(wire
-		(pts
 			(xy 38.735 29.845) (xy 36.195 29.845)
 		)
@@
 	(wire
 		(pts
+			(xy 35.56 77.47) (xy 48.26 77.47)
+		)
+		(stroke
+			(width 0)
+			(type default)
+		)
+	)
+	(wire
+		(pts
 			(xy 99.06 83.82) (xy 111.76 83.82)
 		)
@@
 	(wire
 		(pts
+			(xy 39.37 74.93) (xy 39.37 72.39)
+		)
+		(stroke
+			(width 0)
+			(type default)
+		)
+	)
+	(wire
+		(pts
 			(xy 34.29 100.965) (xy 34.29 103.505)
 		)
@@
 	(wire
 		(pts
-			(xy 43.18 72.39) (xy 114.3 72.39)
+			(xy 144.78 152.4) (xy 144.78 147.32)
 		)
 		(stroke
@@
 	(wire
 		(pts
-			(xy 144.78 152.4) (xy 144.78 147.32)
+			(xy 35.56 74.93) (xy 39.37 74.93)
 		)
 		(stroke
@@
 			)
 		)
-		(property "Footprint" "Connector_PinHeader_2.54mm:PinHeader_1x04_P2.54mm_Vertical"
+		(property "Footprint" "chop_footprint_library:128x64OLED"
 			(at 170.18 147.32 0)
 			(effects
@@
 	(symbol
 		(lib_id "power:GNDREF")
-		(at 43.18 74.93 90)
+		(at 39.37 72.39 90)
 		(unit 1)
 		(exclude_from_sim no)
@@
 		(dnp no)
 		(property "Reference" "#PWR091"
-			(at 49.53 74.93 0)
+			(at 45.72 72.39 0)
 			(effects
 				(font
@@
 		)
 		(property "Value" "GNDREF"
-			(at 46.99 74.93 90)
+			(at 43.18 72.39 90)
 			(effects
 				(font
@@
 		)
 		(property "Footprint" ""
-			(at 43.18 74.93 0)
+			(at 39.37 72.39 0)
 			(effects
 				(font
@@
 		)
 		(property "Datasheet" ""
-			(at 43.18 74.93 0)
+			(at 39.37 72.39 0)
 			(effects
 				(font
@@
 		)
 		(property "Description" ""
-			(at 43.18 74.93 0)
+			(at 39.37 72.39 0)
 			(effects
 				(font
@@
 	)
 	(symbol
-		(lib_id "Connector_Generic:Conn_01x03")
-		(at 38.1 74.93 180)
+		(lib_id "Connector_Generic:Conn_01x02")
+		(at 30.48 77.47 180)
 		(unit 1)
 		(exclude_from_sim no)
@@
 		(dnp no)
 		(property "Reference" "J14"
-			(at 31.115 72.39 0)
+			(at 23.495 74.93 0)
 			(effects
 				(font
@@
 		)
 		(property "Value" "BatteryToMainBoard"
-			(at 31.115 74.93 0)
+			(at 23.495 77.47 0)
 			(effects
 				(font
@@
 			)
 		)
-		(property "Footprint" "Connector_JST:JST_PH_S3B-PH-K_1x03_P2.00mm_Horizontal"
-			(at 38.1 74.93 0)
+		(property "Footprint" "Connector_JST:JST_PH_S2B-PH-K_1x02_P2.00mm_Horizontal"
+			(at 30.48 77.47 0)
 			(effects
 				(font
@@
 		)
 		(property "Datasheet" "~"
-			(at 38.1 74.93 0)
+			(at 30.48 77.47 0)
 			(effects
 				(font
@@
 			)
 		)
-		(property "Description" "Generic connector, single row, 01x03, script generated (kicad-library-utils/schlib/autogen/connector/)"
-			(at 38.1 74.93 0)
+		(property "Description" "Generic connector, single row, 01x02, script generated (kicad-library-utils/schlib/autogen/connector/)"
+			(at 30.48 77.47 0)
 			(effects
 				(font
@@
 		(pin "2"
 		)
-		(pin "3"
-		)
 		(instances

Commit message: Gerber files
Parts:
- added R8: 4.7k, NYSEARCH:R_0603_1608Metric, symbol NYSEARCH:R_Small
Connections:
- net +3.3V: now also R8.1
- net uPC_RTD_DRDY: now reaches J11.9 (Pin_9)
- net uPC_RTD_DRDY: now also U1.25 (33_MCLK2), R8.2
- net HL4_CS renamed uPC_RTD_CS
- net HL4_PWM_IN renamed uPC_PWM_IN
- no-connect marks 30 -> 26
Changed lines of the file:
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@@
 	)
 	(junction
+		(at 34.29 104.14)
+		(diameter 0)
+		(color 0 0 0 0)
+	)
+	(junction
 		(at 109.22 63.5)
 		(diameter 0)
@@
 	)
 	(no_connect
-		(at 187.96 110.49)
-	)
-	(no_connect
 		(at 132.08 85.09)
 	)
@@
 	)
 	(no_connect
-		(at 41.91 55.88)
-	)
-	(no_connect
 		(at 132.08 67.31)
 	)
@@
 	)
 	(no_connect
-		(at 132.08 77.47)
-	)
-	(no_connect
 		(at 102.87 44.45)
 	)
@@
 	)
 	(no_connect
-		(at 132.08 80.01)
-	)
-	(no_connect
 		(at 41.91 58.42)
 	)
@@
 	(wire
 		(pts
+			(xy 34.29 104.14) (xy 43.18 104.14)
+		)
+		(stroke
+			(width 0)
+			(type default)
+		)
+	)
+	(wire
+		(pts
 			(xy 247.65 143.51) (xy 271.78 143.51)
 		)
@@
 	(wire
 		(pts
-			(xy 34.29 103.505) (xy 34.29 109.855)
+			(xy 34.29 103.505) (xy 34.29 104.14)
+		)
+		(stroke
+			(width 0)
+			(type default)
+		)
+	)
+	(wire
+		(pts
+			(xy 34.29 104.14) (xy 34.29 109.855)
 		)
 		(stroke
@@
 		)
 	)
-	(label "HL4_CS"
+	(label "uPC_RTD_CS"
 		(at 132.08 107.95 180)
 		(effects
@@
 		)
 	)
+	(label "uPC_RTD_DRDY"
+		(at 41.91 55.88 0)
+		(effects
+			(font
+				(size 1.27 1.27)
+			)
+			(justify left bottom)
+		)
+	)
 	(label "HL2_CS"
 		(at 29.21 109.855 180)
@@
 		)
 	)
-	(label "HL4_CS"
+	(label "uPC_RTD_CS"
 		(at 29.21 122.555 180)
 		(effects
@@
 		)
 	)
-	(label "HL4_PWM_IN"
+	(label "uPC_PWM_IN"
 		(at 41.91 53.34 0)
 		(effects
@@
 		)
 	)
-	(label "HL4_PWM_IN"
+	(label "uPC_PWM_IN"
 		(at 132.08 64.77 180)
 		(effects
@@
 		)
 	)
-	(label "HL4_CS"
+	(label "uPC_RTD_CS"
 		(at 29.21 55.88 180)
 		(effects
@@
 		)
 	)
+	(label "uPC_RTD_DRDY"
+		(at 187.96 110.49 0)
+		(effects
+			(font
+				(size 1.27 1.27)
+			)
+			(justify left bottom)
+		)
+	)
+	(label "uPC_RTD_DRDY"
+		(at 48.26 104.14 0)
+		(effects
+			(font
+				(size 1.27 1.27)
+			)
+			(justify left bottom)
+		)
+	)
 	(label "SCK_1"
 		(at 41.91 43.18 0)
@@
 					(unit 1)
 				)
+			)
+		)
+	)
+	(symbol
+		(lib_id "NYSEARCH:R_Small")
+		(at 45.72 104.14 90)
+		(unit 1)
+		(exclude_from_sim no)
+		(in_bom yes)
+		(on_board yes)
+		(dnp no)
+		(property "Reference" "R8"
+			(at 45.72 100.33 90)
+			(effects
+				(font
+					(size 1.27 1.27)
+				)
+			)
+		)
+		(property "Value" "4.7k"
+			(at 45.72 102.235 90)
+			(effects
+				(font
+					(size 1.27 1.27)
+				)
+			)
+		)
+		(property "Footprint" "NYSEARCH:R_0603_1608Metric"
+			(at 45.72 104.14 0)
+			(effects
+				(font
+					(size 1.27 1.27)
+				)
+				(hide yes)
+			)
+		)
+		(property "Datasheet" ""
+			(at 45.72 104.14 0)
+			(effects
+				(font
+					(size 1.27 1.27)
+				)
+				(hide yes)
+			)
+		)
+		(property "Description" ""
+			(at 45.72 104.14 0)
+			(effects
+				(font
+					(size 1.27 1.27)
+				)
+			)
+		)
+		(pin "1"
+		)
+		(pin "2"
+		)
+		(instances
+			(project "chop_microcontroller_board"
+				(path "/a68ac1cf-715c-4291-bf7b-de325bf0e054"
+					(reference "R8")
+					(unit 1)
+				)
