File: CHOP_controller_heat/chop-controller-heat.kicad_pcb (KiCad board)
At the start: 4 copper layers, 126.4 x 55.8 mm, 65 parts, among them J1 HL1, J11 SIGNAL1, J12 POWER, J13 TC_SAFETY, J2 HL2, J3 HL3, J4 HL4, K1 J107F1CS1212VDC.36, Q1 DMT6004LPS, Q2 DMT6004LPS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

Commit message: PCB Final 5/24
Parts:
- moved J12 64.5 mm to (139.3, 94.8), turned to 180 degrees
Routing:
- net +24V: track 38.8 -> 0.00 mm
- net +12V: track 43.1 -> 4.89 mm
- net +3.3V: track 78.3 -> 50.8 mm
- net GNDREF: track 175.9 -> 151.2 mm

Commit message: PCB update 5/27
Parts:
- moved J12 66.6 mm to (201.8, 71.8), turned to -90 degrees
Changed lines of the file:
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@@
 	(footprint "Connector_Molex:Molex_Micro-Fit_3.0_43045-0800_2x04_P3.00mm_Horizontal"
 		(layer "F.Cu")
-		(at 139.304 94.8 180)
+		(at 201.804 71.8 -90)
 		(descr "Molex Micro-Fit 3.0 Connector System, 43045-0800 (alternative finishes: 43045-080x), 4 Pins per row (https://www.molex.com/pdm_docs/sd/430450201_sd.pdf), generated with kicad-footprint-generator")
 		(tags "connector Molex Micro-Fit_3.0 horizontal")
 		(property "Reference" "J12"
-			(at 11.6882 2.4696 0)
+			(at 11.6882 2.4696 90)
 			(layer "F.SilkS")
 			(effects
@@
 		)
 		(property "Value" "POWER"
-			(at 4.5 5.7 0)
+			(at 4.5 5.7 90)
 			(layer "F.Fab")
 			(hide yes)
@@
 		)
 		(property "Datasheet" ""
-			(at 0 0 0)
+			(at 0 0 90)
 			(layer "F.Fab")
 			(hide yes)
@@
 		)
 		(property "Description" ""
-			(at 0 0 0)
+			(at 0 0 90)
 			(layer "F.Fab")
 			(hide yes)
@@
 		(attr through_hole)
 		(fp_line
+			(start -3.685 1.1)
+			(end -3.685 -8.03)
+			(stroke
+				(width 0.12)
+				(type solid)
+			)
+			(layer "F.SilkS")
+		)
+		(fp_line
 			(start 12.685 1.1)
 			(end -3.685 1.1)
@@
 		)
 		(fp_line
+			(start -3.685 -8.03)
+			(end -2.685 -9.03)
+			(stroke
+				(width 0.12)
+				(type solid)
+			)
+			(layer "F.SilkS")
+		)
+		(fp_line
 			(start 12.685 -8.03)
 			(end 12.685 1.1)
@@
 		)
 		(fp_line
+			(start -2.685 -9.03)
+			(end 11.685 -9.03)
+			(stroke
+				(width 0.12)
+				(type solid)
+			)
+			(layer "F.SilkS")
+		)
+		(fp_line
 			(start 11.685 -9.03)
 			(end 12.685 -8.03)
@@
 		)
 		(fp_line
-			(start -2.685 -9.03)
-			(end 11.685 -9.03)
-			(stroke
-				(width 0.12)
-				(type solid)
-			)
-			(layer "F.SilkS")
-		)
-		(fp_line
-			(start -3.685 1.1)
-			(end -3.685 -8.03)
-			(stroke
-				(width 0.12)
-				(type solid)
-			)
-			(layer "F.SilkS")
-		)
-		(fp_line
-			(start -3.685 -8.03)
-			(end -2.685 -9.03)
-			(stroke
-				(width 0.12)
-				(type solid)
-			)
-			(layer "F.SilkS")
+			(start -1.25 4.25)
+			(end -1.25 1.5)
+			(stroke
+				(width 0.05)
+				(type solid)
+			)
+			(layer "F.CrtYd")
+		)
+		(fp_line
+			(start 10.25 4.25)
+			(end -1.25 4.25)
+			(stroke
+				(width 0.05)
+				(type solid)
+			)
+			(layer "F.CrtYd")
+		)
+		(fp_line
+			(start -4.08 1.5)
+			(end -4.08 -9.42)
+			(stroke
+				(width 0.05)
+				(type solid)
+			)
+			(layer "F.CrtYd")
+		)
+		(fp_line
+			(start -1.25 1.5)
+			(end -4.08 1.5)
+			(stroke
+				(width 0.05)
+				(type solid)
+			)
+			(layer "F.CrtYd")
+		)
+		(fp_line
+			(start 10.25 1.5)
+			(end 10.25 4.25)
+			(stroke
+				(width 0.05)
+				(type solid)
+			)
+			(layer "F.CrtYd")
 		)
 		(fp_line
@@
 		)
 		(fp_line
+			(start -4.08 -9.42)
+			(end 13.08 -9.42)
+			(stroke
+				(width 0.05)
+				(type solid)
+			)
+			(layer "F.CrtYd")
+		)
+		(fp_line
 			(start 13.08 -9.42)
 			(end 13.08 1.5)
@@
 		)
 		(fp_line
-			(start 10.25 4.25)
-			(end -1.25 4.25)
-			(stroke
-				(width 0.05)
-				(type solid)
-			)
-			(layer "F.CrtYd")
-		)
-		(fp_line
-			(start 10.25 1.5)
-			(end 10.25 4.25)
-			(stroke
-				(width 0.05)
-				(type solid)
-			)
-			(layer "F.CrtYd")
-		)
-		(fp_line
-			(start -1.25 4.25)
-			(end -1.25 1.5)
-			(stroke
-				(width 0.05)
-				(type solid)
-			)
-			(layer "F.CrtYd")
-		)
-		(fp_line
-			(start -1.25 1.5)
-			(end -4.08 1.5)
-			(stroke
-				(width 0.05)
-				(type solid)
-			)
-			(layer "F.CrtYd")
-		)
-		(fp_line
-			(start -4.08 1.5)
-			(end -4.08 -9.42)
-			(stroke
-				(width 0.05)
-				(type solid)
-			)
-			(layer "F.CrtYd")
-		)
-		(fp_line
-			(start -4.08 -9.42)
-			(end 13.08 -9.42)
-			(stroke
-				(width 0.05)
-				(type solid)
-			)
-			(layer "F.CrtYd")
+			(start -3.575 0.99)
+			(end -3.575 -7.92)
+			(stroke
+				(width 0.1)
+				(type solid)
+			)
+			(layer "F.Fab")
+		)
+		(fp_line
+			(start -0.75 0.99)
+			(end 0 0)
+			(stroke
+				(width 0.1)
+				(type solid)
+			)
+			(layer "F.Fab")
 		)
 		(fp_line
@@
 		)
 		(fp_line
+			(start 0 0)
+			(end 0.75 0.99)
+			(stroke
+				(width 0.1)
+				(type solid)
+			)
+			(layer "F.Fab")
+		)
+		(fp_line
+			(start -3.575 -7.92)
+			(end -2.575 -8.92)
+			(stroke
+				(width 0.1)
+				(type solid)
+			)
+			(layer "F.Fab")
+		)
+		(fp_line
 			(start 12.575 -7.92)
 			(end 12.575 0.99)
@@
 		)
 		(fp_line
+			(start -2.575 -8.92)
+			(end 11.575 -8.92)
+			(stroke
+				(width 0.1)
+				(type solid)
+			)
+			(layer "F.Fab")
+		)
+		(fp_line
 			(start 11.575 -8.92)
 			(end 12.575 -7.92)
@@
 			(layer "F.Fab")
 		)
-		(fp_line
-			(start 0 0)
-			(end 0.75 0.99)
-			(stroke
-				(width 0.1)
-				(type solid)
-			)
-			(layer "F.Fab")
-		)
-		(fp_line
-			(start -0.75 0.99)
-			(end 0 0)
-			(stroke
-				(width 0.1)
-				(type solid)
-			)
-			(layer "F.Fab")
-		)
-		(fp_line
-			(start -2.575 -8.92)
-			(end 11.575 -8.92)
-			(stroke
-				(width 0.1)
-				(type solid)
-			)
-			(layer "F.Fab")
-		)
-		(fp_line
-			(start -3.575 0.99)
-			(end -3.575 -7.92)
-			(stroke
-				(width 0.1)
-				(type solid)
-			)
-			(layer "F.Fab")
-		)
-		(fp_line
-			(start -3.575 -7.92)
-			(end -2.575 -8.92)
-			(stroke
-				(width 0.1)
-				(type solid)
-			)
-			(layer "F.Fab")
-		)
 		(fp_text user "${REFERENCE}"
-			(at 4.5 -8.22 0)
+			(at 4.5 -8.22 90)
 			(layer "F.Fab")
 			(effects
@@
 		)
 		(pad "" np_thru_hole circle
-			(at 2.16 -4.32 180)
+			(at 2.16 -4.32 270)
 			(size 3 3)
 			(drill 3)
@@
 		)
 		(pad "" np_thru_hole circle
-			(at 6.86 -4.32 180)
+			(at 6.86 -4.32 270)
 			(size 3 3)
 			(drill 3)
@@
 		)
 		(pad "1" thru_hole roundrect
-			(at 0 0 180)
+			(at 0 0 270)
 			(size 1.5 1.5)
 			(drill 1.02)
@@
 		)
 		(pad "2" thru_hole circle
-			(at 3 0 180)
+			(at 3 0 270)
 			(size 1.5 1.5)
 			(drill 1.02)
@@
 		)
 		(pad "3" thru_hole circle
-			(at 6 0 180)
+			(at 6 0 270)
 			(size 1.5 1.5)
 			(drill 1.02)
@@
 		)
 		(pad "4" thru_hole circle
-			(at 9 0 180)
+			(at 9 0 270)
 			(size 1.5 1.5)
 			(drill 1.02)
@@
 		)
 		(pad "5" thru_hole circle
-			(at 0 3 180)
+			(at 0 3 270)
 			(size 1.5 1.5)
 			(drill 1.02)
@@
 		)
 		(pad "6" thru_hole circle
-			(at 3 3 180)
+			(at 3 3 270)
 			(size 1.5 1.5)
 			(drill 1.02)
@@
 		)
 		(pad "7" thru_hole circle
-			(at 6 3 180)
+			(at 6 3 270)
 			(size 1.5 1.5)
 			(drill 1.02)
@@
 		)
 		(pad "8" thru_hole circle
-			(at 9 3 180)
-			(size 1.5 1.5)
-			(drill 1.02)
+			(at 9 3 270)
+			(size 1.5 1.5)
+			(drill 1.02)
