File: CHOP_controller_heat/chop-controller-heat.kicad_sch (KiCad schematic)
At the start: 11 parts, among them J1 HL1, J11 SIGNAL1, J12 POWER, J13 TC_SAFETY, J2 HL2, J3 HL3, J4 HL4

Commit message: Gerber files
Parts:
- added C29, C30, C36, C37: 100n, NYSEARCH:C_0603_1608Metric_HandSolder, symbol NYSEARCH:C_Small
- added C31, C32, C33, C34: 10n, NYSEARCH:C_0603_1608Metric_HandSolder, symbol NYSEARCH:C_Small
- added C35: 1u, NYSEARCH:C_0603_1608Metric_HandSolder, symbol NYSEARCH:C_Small
- added J9: uPC_RTD, NYSEARCH:Molex_SL_171975-0006_1x06_P2.54mm_Horizontal, symbol Connector_Generic:Conn_01x06
- added R35, R36: 9.53k, NYSEARCH:R_0603_1608Metric, symbol NYSEARCH:R_Small
- added R37, R38: 10.5k, NYSEARCH:R_0603_1608Metric, symbol NYSEARCH:R_Small
- added R39: 10k, NYSEARCH:R_0603_1608Metric, symbol NYSEARCH:R_Small
- added R_REF2: 2k, NYSEARCH:R_0603_1608Metric, symbol NYSEARCH:R_Small
- added U14: ADS1247, Package_SO:TSSOP-20_4.4x6.5mm_P0.65mm, symbol NYSEARCH:ADS1247
Connections:
- net +24V: now also J9.1 (Pin_1)
- net +3.3V: now also C36.1, C37.1, R39.1, U14.1 (DVDD), U14.14 (AVDD), U14.15 (Start)
- net GNDREF: now also C31.1, C32.2, C33.1, C34.1, C35.1, C36.2, C37.2, R36.2, R_REF2.2, U14.13 (AVSS), U14.2 (DGND), U14.3 (CLK), U14.8 (VREFCOM)
- new net: R39.2, U14.4 (N_Reset)
- new net: C35.2, U14.7 (VREFOUT)
- new net MOSFET_uPC: J9.2 (Pin_2)
- new net RTD_MISO: U14.18 (Dout)
- new net RTD_MOSI: U14.19 (DIN)
- new net RTD_SCK: U14.20 (SCLK)
- new net uPC_RTD+: J9.5 (Pin_5), R38.2
- new net uPC_RTD++: J9.6 (Pin_6), U14.12 (AIN3)
- new net uPC_RTD-: J9.4 (Pin_4), R37.2
- new net uPC_RTD--: J9.3 (Pin_3), R35.2, R_REF2.1
- new net uPC_RTD_CS: U14.16 (N_CS)
- new net uPC_RTD_DRDY: U14.17 (N_DRDY)
- new net uPC_RTD_N: C30.1, C33.2, R37.1, U14.10 (AIN1)
- new net uPC_RTD_P: C30.2, C34.2, R38.1, U14.11 (AIN2)
- new net uPC_Ref_N: C29.2, C32.1, R36.1, U14.6 (REFN0)
- new net uPC_Ref_P: C29.1, C31.2, R35.1, U14.5 (REFP0)
- no-connect marks 2 -> 3
