File: CHOP_controller_heat/pwm_heater_drivers.kicad_sch (KiCad schematic)
At the start: 16 parts, among them Q1 DMT6004LPS, Q2 DMT6004LPS, Q6 DMT6004LPS, Q7 DMT6004LPS, U1 TC4427, U2 TC4427

Commit message: Gerber files
Parts:
- removed Q7: DMT6004LPS, NYSEARCH:PowerDI5060-8, symbol NYSEARCH:DMT6004LPS
- removed R12: 100, NYSEARCH:R_0603_1608Metric, symbol NYSEARCH:R_Small
- removed R7: 4.7k, NYSEARCH:R_0603_1608Metric, symbol NYSEARCH:R_Small
- added C4: 1u, NYSEARCH:C_0603_1608Metric_HandSolder, symbol NYSEARCH:C_Small
- added Q9: DMT6004LPS, NYSEARCH:PowerDI5060-8, symbol NYSEARCH:DMT6004LPS
- added R14: 100, NYSEARCH:R_0603_1608Metric, symbol NYSEARCH:R_Small
- added R9: 4.7k, NYSEARCH:R_0603_1608Metric, symbol NYSEARCH:R_Small
- added U4: TC4427, NYSEARCH:MSOP-8_3x3mm_P0.65mm_TI, symbol NYSEARCH:TC4427
Connections:
- net +12V: now also C4.1, U4.6 (Vdd)
- net GNDREF: now also C4.2, Q9.1 (S), R9.2, U4.3 (GND)
- net HL4_PWM_IN: no longer names the net of U2.4 (IN_B)
- new net: Q9.2 (G), R14.1
- new net: R14.2, U4.5 (OUT_B)
- new net MOSFET_uPC: Q9.3 (D)
- new net uPC_PWM_IN: R9.1, U4.4 (IN_B)
- no-connect marks 0 -> 6
Other:
- moved on the sheet: C1, C2, Q1, Q2, Q6, R1, R11, R16, R17, R2, R6, U1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
