File: CHOP_controller_heat/rtd_readout.kicad_sch (KiCad schematic)
At the start: 48 parts, among them U8 ADS1247

Commit message: Gerber files
Parts:
- removed C10 (x2), C20 (x2), C26 (x2), C9 (x2): 100n, NYSEARCH:C_0603_1608Metric_HandSolder, symbol NYSEARCH:C_Small
- removed C11 (x2), C12 (x2), C13 (x2), C14 (x2): 10n, NYSEARCH:C_0603_1608Metric_HandSolder, symbol NYSEARCH:C_Small
- removed C19 (x2): 1u, NYSEARCH:C_0603_1608Metric_HandSolder, symbol NYSEARCH:C_Small
- removed R16 (x2), R17 (x2): 9.53k, NYSEARCH:R_0603_1608Metric, symbol NYSEARCH:R_Small
- removed R18 (x2), R19 (x2): 10.5k, NYSEARCH:R_0603_1608Metric, symbol NYSEARCH:R_Small
- removed R27 (x2): 10k, NYSEARCH:R_0603_1608Metric, symbol NYSEARCH:R_Small
- removed R_REF1 (x2): 2k, NYSEARCH:R_0603_1608Metric, symbol NYSEARCH:R_Small
- removed U8 (x2): ADS1247, Package_SO:TSSOP-20_4.4x6.5mm_P0.65mm, symbol NYSEARCH:ADS1247
- renumbered C9 to C29, C10 to C30, C11 to C31, C12 to C32, C13 to C33, C14 to C34, C19 to C35, C20 to C36, C26 to C37, R16 to R35, R17 to R36, R18 to R37, R19 to R38, R27 to R39, R_REF1 to R_REF2, U8 to U14
Connections:
- no-connect marks 3 -> 1
Other:
- moved on the sheet: C29, C30, C31, C32, C33, C34, C35, C36, C37, R35, R36, R37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
