File: CHOP_controller_heat/safety_cutoff.kicad_sch (KiCad schematic)
At the start: 26 parts, among them K1 J107F1CS1212VDC.36, U16 AD8497, U17 LMC6081, U18 LP2950-3.3_TO92, U19 LMC6081, U20 ADC121S021, U23 NUD3124

Commit message: Gerber files
Parts:
- renumbered C55 to C54, C54 to C55
