File: CHOP_controller_heat/thermocouple_readout.kicad_sch (KiCad schematic)
At the start: 12 parts, among them U10 MAX31855, U11 MAX31855, U6 MAX31855, U7 MAX31855

Commit message: Gerber files
Parts:
- removed C15: 10n, NYSEARCH:C_0603_1608Metric_HandSolder, symbol NYSEARCH:C_Small
- removed C18: 100n, NYSEARCH:C_0603_1608Metric_HandSolder, symbol NYSEARCH:C_Small
- removed U11: MAX31855, NYSEARCH:SO-8_Maxim, symbol NYSEARCH:MAX31855
Other:
- moved on the sheet: C10, C11, C14, C17, C6, C7, U10, U6, U7
